File: main/circuits/CentralBrain/CentralBrain.kicad_pcb (KiCad board)
At the start: 4 copper layers, 46 parts, among them J1 POWER 1234, J2 POWER 5678, J3 POWER 910, J4 EXTRA_TEENSY_PINS, J5 RJ45, J6 TE_5569262-1_08_PORT_RJ45, J7 RJ45_Shielded, J8 AUDIO_PINS, U1 MAX485E, U10 AM26C31CN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

Commit message: lots of work on pcb
Parts:
- moved J4 458.7 mm to (210.2, 104.5)
- moved C6 410.7 mm to (195.0, 49.0)
- moved C4 390.1 mm to (169.0, 50.0)
- moved J8 383.8 mm to (209.2, 79.5)
- moved U3 339.5 mm to (118.0, 84.0)
- moved C2 328.1 mm to (128.0, 51.0)
- moved U5 321.0 mm to (166.2, 98.8)
- moved D10 309.7 mm to (133.0, 158.2), turned to 90 degrees
- moved R9 304.6 mm to (124.0, 149.0), turned to 90 degrees
- moved R7 294.2 mm to (103.0, 150.0), turned to 90 degrees
- moved C3 276.8 mm to (101.0, 50.0)
- moved RV1 276.0 mm to (186.5, 134.5)
- moved RV2 276.0 mm to (201.3, 134.5)
- moved R10 270.3 mm to (133.0, 150.0), turned to 90 degrees
- moved R8 269.9 mm to (111.0, 150.0), turned to 90 degrees
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Connections:
- J5 pad 100: /A-12 -> /A-05
- J5 pad 101: /B-12 -> /B-05
- J5 pad 108: /A-13 -> /A-06
- J5 pad 109: /B-13 -> /B-06
- J5 pad 116: /A-14 -> /A-13
- J5 pad 117: /B-14 -> /B-13
- J5 pad 12: /A-01 -> /A-11
- J5 pad 124: /A-15 -> /A-14
- J5 pad 125: /B-15 -> /B-14
- J5 pad 13: /B-01 -> /B-11
- J5 pad 20: /A-02 -> /A-00
- J5 pad 21: /B-02 -> /B-00
- J5 pad 4: /A-00 -> /A-08
- J5 pad 44: /A-05 -> /A-07
- J5 pad 45: /B-05 -> /B-07
- J5 pad 5: /B-00 -> /B-08
- J5 pad 52: /A-06 -> /A-12
- J5 pad 53: /B-06 -> /B-12
- J5 pad 60: /A-07 -> /A-15
- J5 pad 61: /B-07 -> /B-15
- J5 pad 68: /A-08 -> /A-09
- J5 pad 69: /B-08 -> /B-09
- J5 pad 76: /A-09 -> /A-10
- J5 pad 77: /B-09 -> /B-10
- J5 pad 84: /A-10 -> /A-01
- J5 pad 85: /B-10 -> /B-01
- J5 pad 92: /A-11 -> /A-02
- J5 pad 93: /B-11 -> /B-02
- U3 pad 16: /LED-00 -> /LED-18
- U3 pad 17: /LED-01 -> /LED-19
- U3 pad 18: /LED-02 -> /LED-16
- U3 pad 19: /LED-03 -> /LED-17
- U3 pad 20: /LED-04 -> /LED-14
- U3 pad 21: /LED-05 -> /LED-15
- U3 pad 22: /LED-06 -> /LED-12
- U3 pad 23: /LED-07 -> /LED-13
- U3 pad 24: /LED-08 -> /LED-06
- U3 pad 25: /LED-09 -> /LED-07
- U3 pad 26: /LED-10 -> /LED-04
- U3 pad 27: /LED-11 -> /LED-05
- U3 pad 28: /LED-12 -> /LED-02
- U3 pad 29: /LED-13 -> /LED-03
- U3 pad 30: /LED-14 -> /LED-00
- U3 pad 31: /LED-15 -> /LED-01
- U3 pad 32: /LED-16 -> /LED-10
- U3 pad 33: /LED-17 -> /LED-11
- U3 pad 36: /LED-22 -> /LED-08
- U3 pad 4: /LED-18 -> /LED-22
- U3 pad 44: /LED-23 -> /LED-09
- U3 pad 5: /LED-19 -> /LED-23

Commit message: Mechanical design of PCB mostly done
Parts:
- added H1: MountingHole, MountingHole:MountingHole_3.5mm, F.Cu at (79.0, 93.0)
- added H3: MountingHole, MountingHole:MountingHole_3.5mm, F.Cu at (104.0, 93.0)
- added H4: MountingHole, MountingHole:MountingHole_3.5mm, F.Cu at (185.0, 63.0)
- added H6: MountingHole, MountingHole:MountingHole_3.5mm, F.Cu at (210.0, 63.0)
- J6: footprint Joels KiCad Footprint Library:TE_5569262-1_08_Port_RJ45_New -> Joels KiCad Footprint Library:TE_5569262-1_08_Port_RJ45
- moved J8 181.4 mm to (29.0, 100.0), turned to -90 degrees
- moved RV2 170.6 mm to (39.0, 82.0)
- moved J2 157.8 mm to (238.8, 122.0), turned to 90 degrees
- moved J4 154.0 mm to (59.5, 135.8), turned to 90 degrees
- moved R5 152.1 mm to (232.8, 115.1), turned to 180 degrees
- moved D10 152.0 mm to (230.7, 41.8), turned to -90 degrees
- moved R10 151.6 mm to (233.0, 36.1), turned to 180 degrees
- moved D5 150.7 mm to (231.2, 120.8), turned to -90 degrees
- moved R6 148.5 mm to (232.8, 100.1), turned to 180 degrees
- moved D6 147.1 mm to (231.2, 105.8), turned to -90 degrees
- moved R9 146.5 mm to (233.0, 51.1), turned to 180 degrees
- moved D9 146.2 mm to (230.7, 56.8), turned to -90 degrees
- moved R8 145.9 mm to (233.0, 70.1), turned to 180 degrees
- moved R7 145.2 mm to (232.8, 85.1), turned to 180 degrees
- moved D7 144.8 mm to (231.2, 90.8), turned to -90 degrees
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Connections:
- D10 pad 2: /12V-10 -> /12V_10
- D2 pad 2: /12V-02 -> /12V_02
- D3 pad 2: /12V-03 -> /12V_03
- D4 pad 2: /12V-04 -> /12V_04
- D5 pad 2: /12V-05 -> /12V_05
- D6 pad 2: /12V-06 -> /12V_06
- D7 pad 2: /12V-07 -> /12V_07
- D8 pad 2: /12V-08 -> /12V_08
- D9 pad 2: /12V-09 -> /12V_09
- J1 pad 10: /12V-03 -> /12V_03
- J1 pad 13: /12V-04 -> /12V_04
- J1 pad 14: /12V-04 -> /12V_04
- J1 pad 5: /12V-02 -> /12V_02
- J1 pad 6: /12V-02 -> /12V_02
- J1 pad 9: /12V-03 -> /12V_03
- J2 pad 1: /12V-05 -> /12V_05
- J2 pad 10: /12V-07 -> /12V_07
- J2 pad 13: /12V-08 -> /12V_08
- J2 pad 14: /12V-08 -> /12V_08
- J2 pad 2: /12V-05 -> /12V_05
- J2 pad 5: /12V-06 -> /12V_06
- J2 pad 6: /12V-06 -> /12V_06
- J2 pad 9: /12V-07 -> /12V_07
- J3 pad 1: /12V-09 -> /12V_09
- J3 pad 2: /12V-09 -> /12V_09
- J3 pad 5: /12V-10 -> /12V_10
- J3 pad 6: /12V-10 -> /12V_10
- J4 pad 2: /PIN_10 -> /PIN_1
- J4 pad 3: /PIN_11 -> /PIN_6
- J4 pad 4: /PIN_12 -> /PIN_10
- J4 pad 5: /PIN_15 -> /PIN_11
- J4 pad 6: /PIN_1 -> /PIN_12
- J4 pad 7: /PIN_6 -> /PIN_15
- J5 pad 1: +12V -> /12V_06
- J5 pad 10: +12V -> /12V_05
- J5 pad 105: /12V-07 -> /12V_02
- J5 pad 106: /12V-07 -> /12V_02
- J5 pad 107: /12V-07 -> /12V_02
- J5 pad 11: +12V -> /12V_05
- J5 pad 113: /12V-07 -> /12V_02
- J5 pad 114: /12V-07 -> /12V_02
- J5 pad 115: /12V-07 -> /12V_02
- J5 pad 121: /12V-08 -> +12V
- J5 pad 122: /12V-08 -> +12V
- J5 pad 123: /12V-08 -> +12V
- J5 pad 17: /12V-02 -> /12V_04
- J5 pad 18: /12V-02 -> /12V_04
- J5 pad 19: /12V-02 -> /12V_04
- J5 pad 2: +12V -> /12V_06
- J5 pad 25: /12V-02 -> /12V_03
- J5 pad 26: /12V-02 -> /12V_03
- J5 pad 27: /12V-02 -> /12V_03
- J5 pad 3: +12V -> /12V_06
- J5 pad 33: /12V-03 -> /12V_03
- J5 pad 34: /12V-03 -> /12V_03
- J5 pad 35: /12V-03 -> /12V_03
- J5 pad 41: /12V-03 -> /12V_02
- J5 pad 42: /12V-03 -> /12V_02
- J5 pad 43: /12V-03 -> /12V_02
- J5 pad 49: /12V-04 -> +12V
- J5 pad 50: /12V-04 -> +12V
- J5 pad 51: /12V-04 -> +12V
- J5 pad 57: /12V-04 -> +12V
- J5 pad 58: /12V-04 -> +12V
- J5 pad 59: /12V-04 -> +12V
- J5 pad 65: /12V-05 -> /12V_06
- J5 pad 66: /12V-05 -> /12V_06
- J5 pad 67: /12V-05 -> /12V_06
- J5 pad 73: /12V-05 -> /12V_05
- J5 pad 74: /12V-05 -> /12V_05
- J5 pad 75: /12V-05 -> /12V_05
- J5 pad 81: /12V-06 -> /12V_04
- J5 pad 82: /12V-06 -> /12V_04
- J5 pad 83: /12V-06 -> /12V_04
- J5 pad 89: /12V-06 -> /12V_04
- J5 pad 9: +12V -> /12V_05
- J5 pad 90: /12V-06 -> /12V_04
- J5 pad 91: /12V-06 -> /12V_04
- J5 pad 97: /12V-07 -> /12V_03
- J5 pad 98: /12V-07 -> /12V_03
- J5 pad 99: /12V-07 -> /12V_03
- J6 pad 14: /12V-08 -> /12V_09
- J6 pad 15: /12V-08 -> /12V_09
- J6 pad 16: /12V-08 -> /12V_09
- J6 pad 22: /12V-09 -> /12V_08
- J6 pad 23: /12V-09 -> /12V_08
- J6 pad 24: /12V-09 -> /12V_08
- J6 pad 30: /12V-09 -> /12V_07
- J6 pad 31: /12V-09 -> /12V_07
- J6 pad 32: /12V-09 -> /12V_07
- J6 pad 33: /12V-09 -> /12V_10
- J6 pad 34: /12V-09 -> /12V_10
- J6 pad 35: /12V-09 -> /12V_10
- J6 pad 41: /12V-10 -> /12V_09
- J6 pad 42: /12V-10 -> /12V_09
- J6 pad 43: /12V-10 -> /12V_09
- J6 pad 49: /12V-10 -> /12V_08
- J6 pad 50: /12V-10 -> /12V_08
- J6 pad 51: /12V-10 -> /12V_08
- J6 pad 57: /12V-10 -> /12V_07
- J6 pad 58: /12V-10 -> /12V_07
- J6 pad 59: /12V-10 -> /12V_07
- J6 pad 6: /12V-08 -> /12V_10
- J6 pad 7: /12V-08 -> /12V_10
- J6 pad 8: /12V-08 -> /12V_10
- U3 pad 11: /LED-21 -> /LED-19
- U3 pad 16: /LED-18 -> /LED-20
- U3 pad 17: /LED-19 -> /LED-21
- U3 pad 18: /LED-16 -> /LED-22
- U3 pad 19: /LED-17 -> /LED-23
- U3 pad 20: /LED-14 -> /LED-08
- U3 pad 21: /LED-15 -> /LED-09
- U3 pad 22: /LED-12 -> /LED-10
- U3 pad 23: /LED-13 -> /LED-11
- U3 pad 24: /LED-06 -> /LED-00
- U3 pad 25: /LED-07 -> /LED-01
- U3 pad 26: /LED-04 -> /LED-02
- U3 pad 27: /LED-05 -> /LED-03
- U3 pad 28: /LED-02 -> /LED-04
- U3 pad 29: /LED-03 -> /LED-05
- U3 pad 30: /LED-00 -> /LED-06
- U3 pad 31: /LED-01 -> /LED-07
- U3 pad 32: /LED-10 -> /LED-12
- U3 pad 33: /LED-11 -> /LED-13
- U3 pad 36: /LED-08 -> /LED-14
- U3 pad 4: /LED-22 -> /LED-16
- U3 pad 44: /LED-09 -> /LED-15
- U3 pad 5: /LED-23 -> /LED-17
- U3 pad 6: /LED-20 -> /LED-18
Other:
- board outline added: 238 x 119 mm
- board text added: "30mm^2"
- board text added: "<- WHIPS ANTENNA ->"
