File: main/circuits/CentralBrain/CentralBrain.kicad_sch (KiCad schematic)
At the start: 50 parts, among them J1 POWER 1234, J2 POWER 5678, J3 POWER 910, J4 EXTRA_TEENSY_PINS, J5 RJ45, J6 TE_5569262-1_08_PORT_RJ45, J7 RJ45_Shielded, J8 AUDIO_PINS, U1 MAX485E, U10 AM26C31CN, U11 AM26C31CN, U3 Teensy4.1_Minimal, U4 TSR_1-2450, U5 Teensy4.0_AudioShield_REVD, U6 AM26C31CN, U7 AM26C31CN, U8 AM26C31CN, U9 AM26C31CN

Commit message: version 1.0 of board sent to mfr
Parts:
- added H2: UFO LOGO, Joels KiCad Footprint Library:UFOsmall, symbol Mechanical:MountingHole
Connections:
- net +5V: now also J8.8 (Pin_8)
- net GND: no longer J8.8 (Pin_8)
Changed lines of the file:
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@@
   (junction (at 276.86 111.76) (diameter 0) (color 0 0 0 0)
   )
-  (junction (at 45.72 260.35) (diameter 0) (color 0 0 0 0)
-  )
   (junction (at 138.43 270.51) (diameter 0) (color 0 0 0 0)
   )
@@
   (junction (at 260.35 293.37) (diameter 0) (color 0 0 0 0)
   )
+  (junction (at 52.07 270.51) (diameter 0) (color 0 0 0 0)
+  )
   (junction (at 138.43 293.37) (diameter 0) (color 0 0 0 0)
   )
@@
     (stroke (width 0) (type default) (color 0 0 0 0))
   )
-  (wire (pts (xy 52.07 274.32) (xy 52.07 275.59))
+  (wire (pts (xy 52.07 270.51) (xy 52.07 275.59))
     (stroke (width 0) (type default) (color 0 0 0 0))
   )
@@
     (stroke (width 0) (type default) (color 0 0 0 0))
   )
-  (wire (pts (xy 45.72 260.35) (xy 52.07 260.35))
-    (stroke (width 0) (type default) (color 0 0 0 0))
-  )
   (wire (pts (xy 171.45 311.15) (xy 179.07 311.15))
     (stroke (width 0) (type default) (color 0 0 0 0))
@@
     (stroke (width 0) (type default) (color 0 0 0 0))
   )
+  (wire (pts (xy 52.07 260.35) (xy 52.07 270.51))
+    (stroke (width 0) (type default) (color 0 0 0 0))
+  )
   (wire (pts (xy 147.32 177.8) (xy 160.02 177.8))
     (stroke (width 0) (type default) (color 0 0 0 0))
@@
     (stroke (width 0) (type default) (color 0 0 0 0))
   )
-  (wire (pts (xy 45.72 274.32) (xy 52.07 274.32))
+  (wire (pts (xy 36.83 270.51) (xy 52.07 270.51))
     (stroke (width 0) (type default) (color 0 0 0 0))
   )
@@
     (pin "2")
   )
+  (symbol (lib_id "Mechanical:MountingHole") (at 43.18 332.74 0) (unit 1)
+    (in_bom yes) (on_board yes) (fields_autoplaced)
+    (property "Reference" "H2" (id 0) (at 45.72 331.4699 0)
+      (effects (font (size 1.27 1.27)) (justify left))
+    )
+    (property "Value" "UFO LOGO" (id 1) (at 45.72 334.0099 0)
+      (effects (font (size 1.27 1.27)) (justify left))
+    )
+    (property "Footprint" "Joels KiCad Footprint Library:UFOsmall" (id 2) (at 43.18 332.74 0)
+      (effects (font (size 1.27 1.27)) hide)
+    )
+    (property "Datasheet" "~" (id 3) (at 43.18 332.74 0)
+      (effects (font (size 1.27 1.27)) hide)
+    )
+  )
   (symbol (lib_id "power:GND") (at 340.36 327.66 0) (unit 1)
     (in_bom yes) (on_board yes) (fields_autoplaced)
@@
     (pin "2")
   )
-  (symbol (lib_id "power:+5V") (at 45.72 274.32 0) (unit 1)
-    (in_bom yes) (on_board yes) (fields_autoplaced)
-    (property "Reference" "#PWR0106" (id 0) (at 45.72 278.13 0)
+  (symbol (lib_id "power:+5V") (at 36.83 270.51 0) (unit 1)
+    (in_bom yes) (on_board yes)
+    (property "Reference" "#PWR0106" (id 0) (at 36.83 274.32 0)
       (effects (font (size 1.27 1.27)) hide)
     )
-    (property "Value" "+5V" (id 1) (at 45.72 269.24 0))
-    (property "Footprint" "" (id 2) (at 45.72 274.32 0)
+    (property "Value" "+5V" (id 1) (at 36.83 265.43 0))
+    (property "Footprint" "" (id 2) (at 36.83 270.51 0)
       (effects (font (size 1.27 1.27)) hide)
     )
-    (property "Datasheet" "" (id 3) (at 45.72 274.32 0)
+    (property "Datasheet" "" (id 3) (at 36.83 270.51 0)
       (effects (font (size 1.27 1.27)) hide)
     )
@@
       (reference "H1") (unit 1) (value "MountingHole") (footprint "MountingHole:MountingHole_3.5mm")
     )
+    (path "/33bbea39-d288-4b17-b78b-1b1a8ad9a093"
+      (reference "H2") (unit 1) (value "UFO LOGO") (footprint "Joels KiCad Footprint Library:UFOsmall")
+    )
     (path "/86249b45-c3d8-467c-9fb5-4e6bdfbb6bd6"
